Commit message: add sim branch

File: urdf/jaeger_compl.urdf.xacro (robot description, xacro)
@@ -5,6 +5,6 @@
     <gazebo>
         <plugin
-        filename="ignition-gazebo-odometry-publisher-system"
-        name="ignition::gazebo::systems::OdometryPublisher">
+        filename="gz-sim-odometry-publisher-system"
+        name="gz::sim::systems::OdometryPublisher">
         <odom_publish_frequency>20</odom_publish_frequency>
         <robot_base_frame>base_link</robot_base_frame>
@@ -13,5 +13,5 @@
     </gazebo>
     <gazebo reference="imu_link">
-        <plugin filename="ignition-gazebo-imu-system.so" name="ignition::gazebo::systems::Imu">
+        <plugin filename="gz-sim-imu-system.so" name="gz::sim::systems::Imu">
         </plugin>
         <sensor name="imu_sensor" type="imu">
@@ -77,8 +77,8 @@
         </sensor>
     </gazebo>
-    <!--<gazebo>
+    <!-- <gazebo>
         <plugin
-        filename="ignition-gazebo-joint-state-publisher-system"
-        name="ignition::gazebo::systems::JointStatePublisher">
+        filename="gz-sim-joint-state-publisher-system"
+        name="gz::sim::systems::JointStatePublisher">
         <joint_name>prop1_joint</joint_name>
         <joint_name>prop2_joint</joint_name>
@@ -86,4 +86,32 @@
         <joint_name>prop4_joint</joint_name>
         </plugin>
-    </gazebo>-->
+    </gazebo> -->
+     <ros2_control name="MyRobotHardware" type="system">
+        <hardware>
+          <plugin>jaeger_model/MyRobotHardware</plugin>
+          <parameter name="update_rate" value="50"/>
+        </hardware>
+        <joint name="x_joint">
+          <state_interface name="position"> </state_interface>
+        </joint>
+        <joint name="y_joint">
+          <state_interface name="position"> </state_interface>
+        </joint>
+        <!-- <sensor name="odom_state">
+          <state_interface name="x"/>
+          <state_interface name="y"/>
+        </sensor> -->
+        <gpio name="valve1">
+          <command_interface name="digital"></command_interface>
+        </gpio>
+        <gpio name="valve2">
+          <command_interface name="digital"></command_interface>
+        </gpio>
+        <gpio name="valve3">
+          <command_interface name="digital"></command_interface>
+        </gpio>
+        <gpio name="valve4">
+          <command_interface name="digital"></command_interface>
+        </gpio>
+      </ros2_control>
 </robot>

File: urdf/jaeger_model.urdf (robot description, URDF)
Before this commit: robot jaeger, 12 links, 11 joints
Links:
- removed link prop1_link
- removed link prop2_link
- removed link prop3_link
- removed link prop4_link
- added link valve1, mass 0.02678; collision mesh filename=$(find jaeger_model)/meshes/prop1.STL; visual mesh filename=$(find jaeger_model)/meshes/prop1.STL
- added link valve2, mass 0.02678; collision mesh filename=$(find jaeger_model)/meshes/prop2.STL; visual mesh filename=$(find jaeger_model)/meshes/prop2.STL
- added link valve3, mass 0.02678; collision mesh filename=$(find jaeger_model)/meshes/prop3.STL; visual mesh filename=$(find jaeger_model)/meshes/prop3.STL
- added link valve4, mass 0.02678; collision mesh filename=$(find jaeger_model)/meshes/prop4.STL; visual mesh filename=$(find jaeger_model)/meshes/prop4.STL
- added link x_link, mass 0.001
- added link y_link, mass 0.001
Joints:
- added joint x_joint: type continuous, parent base_link, child x_link, origin xyz=0 0 0 rpy=0 0 0, axis 1 0 0
- added joint y_joint: type continuous, parent base_link, child y_link, origin xyz=0 0 0 rpy=0 0 0, axis 1 0 0
- joint prop1_joint: child prop1_link -> valve1
- joint prop2_joint: child prop2_link -> valve2
- joint prop3_joint: child prop3_link -> valve3
- joint prop4_joint: child prop4_link -> valve4

Commit message: Prueba semifinal

File: urdf/jaeger_compl.urdf.xacro (robot description, xacro)
@@ -77,4 +77,39 @@
         </sensor>
     </gazebo>
+    <gazebo reference="lidar_link">
+      <!-- LiDAR 2D en GPU (puedes cambiar a type='lidar') -->
+      <sensor name="lidar_2d" type="gpu_lidar">
+        <update_rate>20</update_rate>
+        <topic>lidar</topic>  <!-- tópico de Gazebo Transport -->
+        <ray>
+          <scan>
+            <horizontal>
+              <samples>640</samples>
+              <resolution>1</resolution>
+              <min_angle>-3.14159</min_angle>
+              <max_angle> 3.14159</max_angle>
+            </horizontal>
+            <vertical>
+              <samples>1</samples>
+              <resolution>0.01</resolution>
+              <min_angle>0</min_angle>
+              <max_angle>0</max_angle>
+            </vertical>
+          </scan>
+          <range>
+            <min>0.08</min>
+            <max>5.0</max>
+            <resolution>0.01</resolution>
+          </range>
+          <noise>
+            <type>gaussian</type>
+            <mean>0.0</mean>
+            <stddev>0.01</stddev>
+          </noise>
+        </ray>
+        <always_on>1</always_on>
+        <visualize>true</visualize>
+      </sensor>
+    </gazebo>
     <!-- <gazebo>
         <plugin
@@ -90,5 +125,5 @@
         <hardware>
           <plugin>jaeger_model/MyRobotHardware</plugin>
-          <parameter name="update_rate" value="50"/>
+          <parameter name="update_rate" value="100"/>
         </hardware>
         <joint name="x_joint">

File: urdf/jaeger_model.urdf (robot description, URDF)
Before this commit: robot jaeger, 14 links, 13 joints
Links:
- added link lidar_link, mass 0.001; collision cylinder length=0.005 radius=0.01; visual cylinder length=0.005 radius=0.01
Joints:
- added joint lidar_joint: type fixed, parent base_link, child lidar_link, origin xyz=0 0 0.25 rpy=0 0 0

Commit message: Add files via upload

File: urdf/jaeger_compl.urdf.xacro (robot description, xacro)
@@ -1,6 +1,8 @@
 <?xml version="1.0"?>
 <robot xmlns:xacro="http://www.ros.org/wiki/xacro" name="jaeger">
-    <xacro:include filename="$(find jaeger_model)/urdf/jaeger_model.urdf"/>
-    <!-- OdometryPublisher being used instead of Diff Drive's odometry -->
+    <xacro:property name="pkg_share" value="$(find jaeger_model)"/>
+  <!-- Incluye el modelo usando la propiedad -->
+    <xacro:include filename="${pkg_share}/urdf/modelo_tesis.urdf.xacro"/>
+    <!-- OdometryPublisher being used instead of Diff Drive's odometry <xacro:include filename="$(find jaeger_model)/urdf/modelo_tesis.urdf.xacro"/>-->
     <gazebo>
         <plugin

Commit message: cambios finales en doc antes de seguimiento de trayectoria

File: urdf/jaeger_compl.urdf.xacro (robot description, xacro)
@@ -1,6 +1,8 @@
 <?xml version="1.0"?>
 <robot xmlns:xacro="http://www.ros.org/wiki/xacro" name="jaeger">
-    <xacro:include filename="$(find jaeger_model)/urdf/jaeger_model.urdf"/>
-    <!-- OdometryPublisher being used instead of Diff Drive's odometry -->
+    <xacro:property name="pkg_share" value="$(find jaeger_model)"/>
+  <!-- Incluye el modelo usando la propiedad -->
+    <xacro:include filename="${pkg_share}/urdf/Ensamblaje_base2.urdf"/>
+    <!-- OdometryPublisher being used instead of Diff Drive's odometry <xacro:include filename="$(find jaeger_model)/urdf/modelo_tesis.urdf.xacro"/>-->
     <gazebo>
         <plugin
@@ -112,4 +114,8 @@
       </sensor>
     </gazebo>
+    <gazebo reference="base_link">
+      <mu1>0.0034</mu1>
+      <mu2>0.0034</mu2>
+    </gazebo>
     <!-- <gazebo>
         <plugin
@@ -125,5 +131,5 @@
         <hardware>
           <plugin>jaeger_model/MyRobotHardware</plugin>
-          <parameter name="update_rate" value="100"/>
+          <parameter name="update_rate" value="50"/>
         </hardware>
         <joint name="x_joint">
